Commit message: LCS changes

File: robots/youbot.urdf.xacro (robot description, xacro)
@@ -10,4 +10,6 @@
   <!-- youbot base -->
   <xacro:include filename="$(find youbot_description)/urdf/youbot_base/base.urdf.xacro" />
+  <!-- youbot camera -->
+  <xacro:include filename="$(find youbot_description)/urdf/sensors/microsoft_lifecam.urdf.xacro" />
   <!-- youbot plate -->
   <xacro:include filename="$(find youbot_description)/urdf/youbot_plate/plate.urdf.xacro" />
@@ -20,6 +22,10 @@
   <!-- materials for visualization -->
   <xacro:include filename="$(find youbot_description)/urdf/materials.urdf.xacro" />
+  <!-- kinect camera for image and deph visualization-->
+  <xacro:include filename="$(find youbot_description)/urdf/sensors/kinect_camera.urdf.xacro" />
+    <!-- kinect camera 2 for second image and deph visualization-->
+  <xacro:include filename="$(find youbot_description)/urdf/sensors/kinect_camera2.urdf.xacro" />
   <!-- sensors -->
-  <xacro:include filename="$(find youbot_description)/urdf/sensors/hokuyo_urg04_laser.urdf.xacro"/>
+  <!-- <xacro:include filename="$(find youbot_description)/urdf/sensors/hokuyo_urg04_laser.urdf.xacro"/> -->
   <!-- Now we can start using the macros xacro:included above to define the actual youbot -->
   <!-- The first use of a macro.  This one was defined in base.urdf.xacro above.
@@ -41,7 +47,15 @@
     <origin xyz="0 0 0" rpy="0 0 0" />
   </xacro:youbot_gripper>
+  <!-- kinect camera -->
+  <xacro:kinect_camera name="camera_endpoint" parent="arm_link_5" ros_topic="base_scan" update_rate="10" min_angle="-1.57" max_angle="1.57">
+    <origin xyz="-0.08 0 0.03" rpy="0 4.71239 0" />
+  </xacro:kinect_camera>
+  <!-- kinect second camera -->
+  <xacro:kinect_camera2 name="camera2" parent="base_link" ros_topic="base_scan" update_rate="10" min_angle="-1.57" max_angle="1.57">
+    <origin xyz="0.35 0 0.085" rpy="0 0 0" />
+  </xacro:kinect_camera2>
   <!-- base laser front -->
-  <xacro:hokuyo_urg04_laser name="base_laser_front" parent="base" ros_topic="base_scan" update_rate="10" min_angle="-1.57" max_angle="1.57">
+  <!-- <xacro:hokuyo_urg04_laser name="base_laser_front" parent="base" ros_topic="base_scan" update_rate="10" min_angle="-1.57" max_angle="1.57">
     <origin xyz="0.3 0 -0.03" rpy="0 0 0"/>
-  </xacro:hokuyo_urg04_laser>
+  </xacro:hokuyo_urg04_laser> -->
 </robot>

File: urdf/sensors/kinect_camera.gazebo.xacro (robot description, xacro)
@@ -1,57 +1,79 @@
 <?xml version="1.0"?>
-<root xmlns:sensor="http://playerstage.sourceforge.net/gazebo/xmlschema/#sensor"
-      xmlns:controller="http://playerstage.sourceforge.net/gazebo/xmlschema/#controller"
-      xmlns:interface="http://playerstage.sourceforge.net/gazebo/xmlschema/#interface"
-      xmlns:xacro="http://ros.org/wiki/xacro">
-<xacro:macro name="kinect_camera_gazebo" params="name">
-  <gazebo reference="${name}_camera">
-    <sensor:camera name="${name}_depth_frame_sensor">
-      <imageFormat>R8G8B8</imageFormat>
-      <imageSize>640 480</imageSize>
-      <hfov>57</hfov>
-      <nearClip>0.01</nearClip>
-      <farClip>5</farClip>
-      <updateRate>20.0</updateRate>
-      <baseline>0.2</baseline>
-      <controller:gazebo_ros_camera name="${name}_depth_frame_controller" plugin="libgazebo_ros_camera.so">
-        <alwaysOn>true</alwaysOn>
-        <updateRate>20.0</updateRate>
-        <imageTopicName>/camera/ir/image_raw</imageTopicName>
-        <cameraInfoTopicName>/camera/ir/camera_info</cameraInfoTopicName>
-        <depthImageTopicName>/camera/depth/image_raw</depthImageTopicName>
-        <depthImageInfoTopicName>/camera/depth/camera_info</depthImageInfoTopicName>
-        <pointCloudTopicName>/camera/depth/points</pointCloudTopicName>
-        <frameName>/${name}_depth_optical_frame</frameName>
-        <pointCloudCutoff>0.5</pointCloudCutoff>
-        <distortion_k1>0.00000001</distortion_k1>
-        <distortion_k2>0.00000001</distortion_k2>
-        <distortion_k3>0.00000001</distortion_k3>
-        <distortion_t1>0.00000001</distortion_t1>
-        <distortion_t2>0.00000001</distortion_t2>
-      </controller:gazebo_ros_camera>
-    </sensor:camera>
-    <sensor:camera name="${name}_rgb_frame_sensor">
-      <imageFormat>R8G8B8</imageFormat>
-      <imageSize>640 480</imageSize>
-      <hfov>57</hfov>
-      <nearClip>0.01</nearClip>
-      <farClip>5</farClip>
-      <updateRate>20.0</updateRate>
-      <baseline>0.2</baseline>
-      <controller:gazebo_ros_camera name="${name}_rgb_frame_controller" plugin="libgazebo_ros_camera.so">
-        <alwaysOn>true</alwaysOn>
-        <updateRate>20.0</updateRate>
-        <imageTopicName>/camera/rgb/image_raw</imageTopicName>
-        <cameraInfoTopicName>/camera/rgb/camera_info</cameraInfoTopicName>
-        <frameName>/${name}_rgb_optical_frame</frameName>
-        <pointCloudCutoff>0.5</pointCloudCutoff>
-        <distortion_k1>0.00000001</distortion_k1>
-        <distortion_k2>0.00000001</distortion_k2>
-        <distortion_k3>0.00000001</distortion_k3>
-        <distortion_t1>0.00000001</distortion_t1>
-        <distortion_t2>0.00000001</distortion_t2>
-      </controller:gazebo_ros_camera>
-    </sensor:camera>
-  </gazebo>
-</xacro:macro>
-</root>
+<robot xmlns:sensor="http://playerstage.sourceforge.net/gazebo/xmlschema/#sensor"
+       xmlns:controller="http://playerstage.sourceforge.net/gazebo/xmlschema/#controller"
+       xmlns:interface="http://playerstage.sourceforge.net/gazebo/xmlschema/#interface"
+       xmlns:xacro="http://ros.org/wiki/xacro">
+  <xacro:macro name="kinect_camera_gazebo" params="name ros_topic update_rate min_angle max_angle">
+    <!-- <gazebo reference="${name}_link"> -->
+    <gazebo reference="${name}">
+      <sensor name="${name}" type="ray">
+		<always_on>true</always_on>
+        <update_rate>${update_rate}</update_rate>
+		<pose>0 0 0 0 0 0</pose>
+		<visualize>false</visualize>
+        <ray>
+            <scan>
+                <horizontal>
+                    <samples>150</samples>
+                    <resolution>1.0</resolution>
+                    <min_angle>${min_angle}</min_angle>
+                    <max_angle>${max_angle}</max_angle>
+                </horizontal>
+            </scan>
+            <range>
+				<min>0.05</min>
+				<max>5.6</max>
+				<resolution>0.36</resolution>
+			</range>
+        </ray>
+        <plugin name="gazebo_ros_${name}_controller" filename="libgazebo_ros_laser.so">
+            <gaussianNoise>0.005</gaussianNoise>
+            <alwaysOn>true</alwaysOn>
+            <updateRate>${update_rate}</updateRate>
+            <topicName>${ros_topic}</topicName>
+            <!-- <frameName>/${name}_link</frameName> -->
+            <frameName>/${name}</frameName>
+         </plugin>
+      </sensor>
+      <sensor name="camera" type="depth">
+        <camera>
+          <horizontal_fov>1.04719755</horizontal_fov>
+          <image>
+            <width>640</width>
+            <height>480</height>
+          </image>
+          <clip>
+            <near>0.1</near>
+            <far>20</far>
+          </clip>
+        </camera>
+        <plugin name="camera_plugin" filename="libgazebo_ros_openni_kinect.so">
+          <baseline>0.2</baseline>
+          <alwaysOn>true</alwaysOn>
+          <!-- Keep this zero, update_rate in the parent <sensor> tag
+            will control the frame rate. -->
+          <updateRate>0.0</updateRate>
+          <cameraName>camera_ir</cameraName>
+          <imageTopicName>/camera/color/image_raw</imageTopicName>
+          <cameraInfoTopicName>/camera/color/camera_info</cameraInfoTopicName>
+          <depthImageTopicName>/camera/depth/image_raw</depthImageTopicName>
+          <depthImageCameraInfoTopicName>/camera/depth/camera_info</depthImageCameraInfoTopicName>
+          <pointCloudTopicName>/camera/depth/points</pointCloudTopicName>
+          <frameName>camera_link</frameName>
+          <pointCloudCutoff>0.5</pointCloudCutoff>
+          <pointCloudCutoffMax>3.0</pointCloudCutoffMax>
+          <distortionK1>0</distortionK1>
+          <distortionK2>0</distortionK2>
+          <distortionK3>0</distortionK3>
+          <distortionT1>0</distortionT1>
+          <distortionT2>0</distortionT2>
+          <CxPrime>0</CxPrime>
+          <Cx>0</Cx>
+          <Cy>0</Cy>
+          <focalLength>0</focalLength>
+          <hackBaseline>0</hackBaseline>
+        </plugin>
+      </sensor>
+    </gazebo>
+  </xacro:macro>
+</robot>

File: urdf/sensors/kinect_camera.urdf.xacro (robot description, xacro)
@@ -1,93 +1,41 @@
 <?xml version="1.0"?>
-<root xmlns:sensor="http://playerstage.sourceforge.net/gazebo/xmlschema/#sensor"
-      xmlns:controller="http://playerstage.sourceforge.net/gazebo/xmlschema/#controller"
-      xmlns:interface="http://playerstage.sourceforge.net/gazebo/xmlschema/#interface"
-      xmlns:xacro="http://ros.org/wiki/xacro">
-  <xacro:include filename="$(find youbot_description)/urdf/sensors/kinect_camera.gazebo.xacro"/>
-  <xacro:macro name="kinect_camera" params="name parent *origin">
-   <joint name="${name}_camera_joint" type="fixed">
-    <xacro:insert_block name="origin" />
-    <parent link="${parent}" />
-    <child link="${name}_camera" />
-   </joint>
-   <link name="${name}_camera">
-    <inertial>
-      <mass value="0.01" />
-      <origin xyz="0 0 0" />
-      <inertia ixx="0.001" ixy="0.0" ixz="0.0"
-        iyy="0.001" iyz="0.0"
-        izz="0.001" />
-    </inertial>
-    <visual>
-      <origin xyz="0.0 0.0 0.0" rpy="0 0 0" />
-      <geometry>
-       <mesh filename="package://youbot_description/meshes/sensors/kinect.dae"/>
-      </geometry>
-    </visual>
-    <collision>
-      <origin xyz="0.0 0.0 0.0" rpy="0 0 0" />
-      <geometry>
-        <mesh filename="package://youbot_description/meshes/sensors/kinect.dae"/>
-      </geometry>
-    </collision>
-  </link>
-  <joint name="${name}_camera_depth_joint" type="fixed">
-    <origin xyz="0 0.018 0" rpy="0 0 0" />
-    <parent link="${name}_camera" />
-    <child link="${name}_depth_frame" />
-  </joint>
-  <link name="${name}_depth_frame">
-    <inertial>
-      <mass value="0.01" />
-      <origin xyz="0 0 0" />
-      <inertia ixx="0.001" ixy="0.0" ixz="0.0"
-        iyy="0.001" iyz="0.0"
-        izz="0.001" />
-    </inertial>
-  </link>
-  <joint name="${name}_camera_depth_optical_joint" type="fixed">
-    <origin xyz="0 0 0" rpy="${-M_PI/2} 0 ${-M_PI/2}" />
-    <parent link="${name}_depth_frame" />
-    <child link="${name}_depth_optical_frame" />
-  </joint>
-  <link name="${name}_depth_optical_frame">
-    <inertial>
-      <mass value="0.001" />
-      <origin xyz="0 0 0" />
-      <inertia ixx="0.0001" ixy="0.0" ixz="0.0"
-        iyy="0.0001" iyz="0.0"
-        izz="0.0001" />
-    </inertial>
-  </link>
-  <joint name="${name}_camera_rgb_joint" type="fixed">
-    <origin xyz="0 -0.005 0" rpy="0 0 0" />
-    <parent link="${name}_camera" />
-    <child link="${name}_rgb_frame" />
-  </joint>
-  <link name="${name}_rgb_frame">
-    <inertial>
-      <mass value="0.001" />
-      <origin xyz="0 0 0" />
-      <inertia ixx="0.0001" ixy="0.0" ixz="0.0"
-        iyy="0.0001" iyz="0.0"
-        izz="0.0001" />
-    </inertial>
-  </link>
-  <joint name="${name}_camera_rgb_optical_joint" type="fixed">
-    <origin xyz="0 0 0" rpy="${-M_PI/2} 0 ${-M_PI/2}" />
-    <parent link="${name}_rgb_frame" />
-    <child link="${name}_rgb_optical_frame" />
-  </joint>
-  <link name="${name}_rgb_optical_frame">
-    <inertial>
-      <mass value="0.001" />
-      <origin xyz="0 0 0" />
-      <inertia ixx="0.0001" ixy="0.0" ixz="0.0"
-        iyy="0.0001" iyz="0.0"
-        izz="0.0001" />
-    </inertial>
-  </link>
-  <!-- for simulation -->
-  <xacro:kinect_camera_gazebo name="openni" />
-</xacro:macro>
-</root>
+<robot xmlns:sensor="http://playerstage.sourceforge.net/gazebo/xmlschema/#sensor"
+       xmlns:controller="http://playerstage.sourceforge.net/gazebo/xmlschema/#controller"
+       xmlns:interface="http://playerstage.sourceforge.net/gazebo/xmlschema/#interface"
+       xmlns:xacro="http://ros.org/wiki/xacro">
+  <xacro:include filename="$(find youbot_description)/urdf/sensors/kinect_camera.gazebo.xacro" />
+  <!-- <xacro:include filename="$(find youbot_description)/urdf/sensors/kinect_camera2.gazebo.xacro" /> -->
+  <xacro:macro name="kinect_camera" params="name parent *origin ros_topic update_rate min_angle max_angle">
+    <joint name="${name}_hokuyo_urg04_laser_joint" type="fixed">
+      <axis xyz="0 1 0" />
+      <xacro:insert_block name="origin" />
+      <!-- <parent link="${parent}_link"/> -->
+      <parent link="${parent}"/>
+      <!-- <child link="${name}_link"/> -->
+      <child link="${name}"/>
+    </joint>
+    <!-- <link name="${name}_link" type="laser"> -->
+    <link name="${name}" type="laser">
+      <inertial>
+        <mass value="0.16" />
+        <origin xyz="0 0 0" rpy="0 0 0" />
+        <inertia ixx="0.1" ixy="0" ixz="0" iyy="0.1" iyz="0" izz="0.1" />
+      </inertial>
+      <visual>
+      	<origin xyz="0 0 0" rpy="0 0 0" />
+	<geometry>
+    <mesh filename="package://youbot_description/meshes/sensors/kinect.dae"/>
+	</geometry>
+	<material name="DarkGrey" />
+      </visual>
+      <collision>
+		<origin xyz="0 0 0" rpy="0 0 0" />
+		<geometry>
+      <mesh filename="package://youbot_description/meshes/sensors/kinect.dae"/>
+		</geometry>
+	</collision>
+    </link>
+    <!-- gazebo extensions -->
+    <xacro:kinect_camera_gazebo name="${name}" ros_topic="${ros_topic}" update_rate="${update_rate}" min_angle="${min_angle}" max_angle="${max_angle}" />
+  </xacro:macro>
+</robot>
